File: pcbs/eom_test_pcb/eom_test_pcb.brd (EAGLE design)
At the start: 160 x 47.9 mm, 72 parts

Commit message: commit before restart
Parts:
- moved X7 59.5 mm to (51.9, 98.6), turned to 270 degrees
- moved X11 59.3 mm to (108.7, 98.8), turned to 270 degrees
- moved X17 44.7 mm to (153.1, 98.8)
- moved X1 44.4 mm to (7.49, 98.7)
- moved X6 40.5 mm to (40.8, 98.6), turned to 270 degrees
- moved X12 40.2 mm to (119.9, 98.9), turned to 270 degrees
- moved X3 30.1 mm to (1.32, 89.2), turned to 0 degrees
- moved X15 29.6 mm to (159.0, 89.1), turned to 180 degrees
- moved X2 22.4 mm to (18.6, 98.7)
- moved X16 22.4 mm to (142.1, 98.8)
- moved X18 21.4 mm to (159.0, 78.3), turned to 180 degrees
- moved X5 21.1 mm to (1.21, 78.5), turned to 0 degrees
- moved X13 11.0 mm to (158.9, 67.2)
- moved X14 11.0 mm to (131.0, 98.8)
- moved X4 10.9 mm to (29.6, 98.6)
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Routing:
- net N$33: track 39.6 -> 78.2 mm
- net N$13: track 80.9 -> 42.6 mm
- net N$1: track 40.0 -> 73.1 mm
- net N$21: track 79.3 -> 47.5 mm
- net N$11: track 73.6 -> 49.6 mm
- net N$3: track 43.9 -> 67.4 mm
- net N$31: track 45.9 -> 68.9 mm
- net N$23: track 75.7 -> 55.7 mm
- net N$29: track 57.5 -> 77.2 mm
- net N$5: track 54.4 -> 73.3 mm
- net N$27: track 68.6 -> 60.2 mm
- net N$9: track 77.3 -> 69.5 mm
- net N$7: track 66.0 -> 59.0 mm
- net N$35: track 77.1 -> 72.1 mm
- net N$25: track 73.9 -> 78.1 mm
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
Commit message: commit before going downstairs to meet with Luis
Parts:
- moved R12 19.8 mm to (126.3, 60.3)
- moved R18 19.8 mm to (129.5, 60.3)
- moved R10 19.8 mm to (123.2, 60.3)
- moved R11 19.8 mm to (116.8, 60.3)
- moved R13 19.8 mm to (113.7, 60.3)
- moved R14 19.8 mm to (120.0, 60.3)
- moved R15 19.8 mm to (110.6, 60.3)
- moved R16 19.8 mm to (132.6, 60.3)
- moved R17 19.8 mm to (107.5, 60.3)
- moved R6 17.2 mm to (29.9, 60.3)
- moved R1 17.2 mm to (42.5, 60.3)
- moved R2 17.2 mm to (36.2, 60.3)
- moved R3 17.2 mm to (45.7, 60.3)
- moved R4 17.2 mm to (39.4, 60.3)
- moved R5 17.2 mm to (48.9, 60.3)
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Routing:
- net N$19: track 87.9 -> 0.00 mm
- net N$33: track 78.2 -> 0.00 mm
- net N$25: track 78.1 -> 0.00 mm
- net N$29: track 77.2 -> 0.00 mm
- net N$35: track 72.1 -> 0.00 mm
- net N$31: track 68.9 -> 0.00 mm
- net N$27: track 60.2 -> 0.00 mm
- net N$23: track 55.7 -> 0.00 mm
- net GND: track 50.5 -> 0.00 mm
- net N$21: track 47.5 -> 0.00 mm
- net N$18: track 40.8 -> 0.00 mm
- net N$32: track 37.8 -> 0.00 mm
- net N$12: track 36.6 -> 0.00 mm
- net N$36: track 33.7 -> 0.00 mm
- net N$24: track 29.9 -> 0.00 mm
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Other:
- board size 160 x 47.9 mm -> 160 x 48 mm
