File: pcbs/eom_test_pcb_v2/eom_test_pcb_v2.brd (EAGLE design)
At the start: 98.3 x 23 mm, 32 parts, among them J1 142-0711-821, J2 142-0711-821, J3 142-0711-821, J4 142-0711-821, J5 142-0711-821, J6 142-0711-821, J7 142-0711-821, J8 142-0711-821

Commit message: quarter way done with routing
Parts:
- added JP1: (no value), adafruit:1X03
- added R10, R9: (no value), adafruit:R0402
- moved R7 136.7 mm to (64.1, 78.5), turned to 180 degrees
- moved R8 132.1 mm to (64.1, 76.0), turned to 180 degrees
- moved R6 126.7 mm to (41.3, 76.0), turned to 180 degrees
- moved R5 111.1 mm to (48.9, 78.5), turned to 180 degrees
- moved U$7 110.1 mm to (72.1, 74.4), turned to 90 degrees
- moved U$8 109.8 mm to (72.1, 75.9), turned to 90 degrees
- moved J2 107.2 mm to (134.9, 90.4), turned to 0 degrees
- moved R4 105.0 mm to (56.6, 75.9), turned to 180 degrees
- moved U$6 98.0 mm to (72.1, 78.3), turned to 90 degrees
- moved U$5 97.5 mm to (72.1, 75.1), turned to 90 degrees
- moved J3 94.5 mm to (122.2, 63.8), turned to 180 degrees
- moved R3 92.3 mm to (56.6, 78.5), turned to 180 degrees
- moved J4 91.2 mm to (134.9, 63.8)
- moved U$3 88.8 mm to (72.1, 79.1), turned to 90 degrees
- moved U$4 87.8 mm to (72.1, 80.5), turned to 90 degrees
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Connections:
- removed net N$10: R5.1, U$10.P$1
- removed net N$11: J6.1, U$11.P$1
- removed net N$12: R6.1, U$12.P$1
- removed net N$13: J7.1, U$13.P$1
- removed net N$14: R7.1, U$14.P$1
- removed net N$15: J8.1, U$15.P$1
- removed net N$16: R8.1, U$16.P$1
- removed net N$8: R4.1, U$8.P$1
- removed net N$9: J5.1, U$9.P$1
- new net TM1: JP1.3, R9.1
- new net TM2: JP1.1, R10.1
- net GND: now also JP1.2, R10.2, R9.2
- net N$1: now also R7.1, U$6.P$1; no longer J1.1, U$1.P$1
- net N$2: now also R8.1, U$8.P$1; no longer R1.1, U$2.P$1
- net N$3: now also R3.1; no longer J2.1
- net N$4: now also R4.1, U$5.P$1; no longer R2.1, U$4.P$1
- net N$5: now also R5.1, U$1.P$1; no longer J3.1, U$5.P$1
- net N$6: now also R2.1, U$7.P$1; no longer R3.1, U$6.P$1
- net N$7: now also R1.1, U$4.P$1; no longer J4.1, U$7.P$1
Routing:
- net N$7: track 0.00 -> 31.4 mm
- net N$5: track 0.00 -> 23.1 mm
- net N$3: track 0.00 -> 15.1 mm
- net N$1: track 0.00 -> 6.74 mm
Other:
- board size 98.3 x 23 mm -> 116.1 x 23 mm
