File: pcbs/eom_test_pcb_v2/eom_test_pcb_v2.brd (EAGLE design)
At the start: 127.2 x 23.4 mm, 35 parts, among them J1 142-0711-821, J2 142-0711-821, J3 142-0711-821, J4 142-0711-821, J5 142-0711-821, J6 142-0711-821, J7 142-0711-821, J8 142-0711-821

Commit message: Adjusted traces to 6.8mil and fixed DRC complaints
Routing:
- net GND: vias 864 -> 863
