File: pcbs/eom_test_pcb_v2/eom_test_pcb_v2.sch (EAGLE design)
At the start: 32 parts, among them J1 142-0711-821, J2 142-0711-821, J3 142-0711-821, J4 142-0711-821, J5 142-0711-821, J6 142-0711-821, J7 142-0711-821, J8 142-0711-821

Commit message: quarter way done with routing
Parts:
- added JP1: (no value), adafruit:PINHD-1X3
- added R10, R9: (no value), adafruit:R-US_R0402
Connections:
- removed net N$10: R5.1, U$10.P$1
- removed net N$11: J6.1, U$11.P$1
- removed net N$12: R6.1, U$12.P$1
- removed net N$13: J7.1, U$13.P$1
- removed net N$14: R7.1, U$14.P$1
- removed net N$15: J8.1, U$15.P$1
- removed net N$16: R8.1, U$16.P$1
- removed net N$8: R4.1, U$8.P$1
- removed net N$9: J5.1, U$9.P$1
- new net TM1: JP1.3, R9.1
- new net TM2: JP1.1, R10.1
- net GND: now also JP1.2, R10.2, R9.2
- net N$1: now also R7.1, U$6.P$1; no longer J1.1, U$1.P$1
- net N$2: now also R8.1, U$8.P$1; no longer R1.1, U$2.P$1
- net N$3: now also R3.1; no longer J2.1
- net N$4: now also R4.1, U$5.P$1; no longer R2.1, U$4.P$1
- net N$5: now also R5.1, U$1.P$1; no longer J3.1, U$5.P$1
- net N$6: now also R2.1, U$7.P$1; no longer R3.1, U$6.P$1
- net N$7: now also R1.1, U$4.P$1; no longer J4.1, U$7.P$1
Changed lines of the file:
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@@
 <part name="R8" library="adafruit" deviceset="R-US_" device="M1206" package3d_urn="urn:adsk.eagle:package:6240588/1"/>
 <part name="J8" library="eom_chip_lib" deviceset="142-0711-821" device=""/>
+<part name="R9" library="adafruit" library_urn="urn:adsk.eagle:library:420" deviceset="R-US_" device="R0402" package3d_urn="urn:adsk.eagle:package:6240564/1"/>
+<part name="R10" library="adafruit" library_urn="urn:adsk.eagle:library:420" deviceset="R-US_" device="R0402" package3d_urn="urn:adsk.eagle:package:6240564/1"/>
+<part name="JP1" library="adafruit" library_urn="urn:adsk.eagle:library:420" deviceset="PINHD-1X3" device="" package3d_urn="urn:adsk.eagle:package:6240710/1"/>
 </parts>
 <sheets>
@@
 <attribute name="NAME" x="143.1544" y="15.0114" size="2.0828" layer="95" ratio="6" rot="SR180"/>
 </instance>
+<instance part="R9" gate="G$1" x="81.28" y="-2.54" smashed="yes">
+<attribute name="NAME" x="77.47" y="-1.0414" size="1.778" layer="95"/>
+<attribute name="VALUE" x="77.47" y="-5.842" size="1.778" layer="96"/>
+</instance>
+<instance part="R10" gate="G$1" x="180.34" y="-2.54" smashed="yes">
+<attribute name="NAME" x="176.53" y="-1.0414" size="1.778" layer="95"/>
+<attribute name="VALUE" x="176.53" y="-5.842" size="1.778" layer="96"/>
+</instance>
+<instance part="JP1" gate="A" x="132.08" y="-22.86" smashed="yes" rot="R270">
+<attribute name="NAME" x="137.795" y="-16.51" size="1.778" layer="95" rot="R270"/>
+<attribute name="VALUE" x="124.46" y="-16.51" size="1.778" layer="96" rot="R270"/>
+</instance>
 </instances>
 <busses>
 </busses>
 <nets>
-<net name="N$1" class="0">
-<segment>
-<pinref part="U$1" gate="G$1" pin="P$1"/>
-<wire x1="67.31" y1="68.58" x2="48.26" y2="68.58" width="0.1524" layer="91"/>
-<pinref part="J1" gate="A" pin="1"/>
-</segment>
-</net>
-<net name="N$2" class="0">
-<segment>
-<pinref part="U$2" gate="G$1" pin="P$1"/>
-<pinref part="R1" gate="G$1" pin="1"/>
-<wire x1="95.25" y1="68.58" x2="104.14" y2="68.58" width="0.1524" layer="91"/>
-</segment>
-</net>
 <net name="GND" class="0">
 <segment>
@@
 <label x="152.4" y="25.4" size="1.778" layer="95"/>
 </segment>
+<segment>
+<pinref part="R9" gate="G$1" pin="2"/>
+<label x="91.44" y="-2.54" size="1.778" layer="95"/>
+<pinref part="JP1" gate="A" pin="2"/>
+<wire x1="86.36" y1="-2.54" x2="132.08" y2="-2.54" width="0.1524" layer="91"/>
+<wire x1="132.08" y1="-2.54" x2="132.08" y2="-20.32" width="0.1524" layer="91"/>
+</segment>
+<segment>
+<pinref part="R10" gate="G$1" pin="2"/>
+<wire x1="185.42" y1="-2.54" x2="195.58" y2="-2.54" width="0.1524" layer="91"/>
+<label x="190.5" y="-2.54" size="1.778" layer="95"/>
+</segment>
+</net>
+<net name="TM1" class="0">
+<segment>
+<pinref part="JP1" gate="A" pin="3"/>
+<wire x1="129.54" y1="-20.32" x2="71.12" y2="-20.32" width="0.1524" layer="91"/>
+<pinref part="R9" gate="G$1" pin="1"/>
+<wire x1="71.12" y1="-20.32" x2="71.12" y2="-2.54" width="0.1524" layer="91"/>
+<wire x1="71.12" y1="-2.54" x2="76.2" y2="-2.54" width="0.1524" layer="91"/>
+<label x="76.2" y="-20.32" size="1.778" layer="95"/>
+</segment>
+</net>
+<net name="TM2" class="0">
+<segment>
+<pinref part="JP1" gate="A" pin="1"/>
+<pinref part="R10" gate="G$1" pin="1"/>
+<wire x1="134.62" y1="-20.32" x2="175.26" y2="-20.32" width="0.1524" layer="91"/>
+<wire x1="175.26" y1="-20.32" x2="175.26" y2="-2.54" width="0.1524" layer="91"/>
+<label x="154.94" y="-20.32" size="1.778" layer="95"/>
+</segment>
+</net>
+<net name="N$1" class="0">
+<segment>
+<pinref part="U$6" gate="G$1" pin="P$1"/>
+<wire x1="95.25" y1="35.56" x2="99.06" y2="35.56" width="0.1524" layer="91"/>
+<wire x1="99.06" y1="35.56" x2="99.06" y2="93.98" width="0.1524" layer="91"/>
+<wire x1="99.06" y1="93.98" x2="198.12" y2="93.98" width="0.1524" layer="91"/>
+<wire x1="198.12" y1="93.98" x2="198.12" y2="35.56" width="0.1524" layer="91"/>
+<pinref part="R7" gate="G$1" pin="1"/>
+<wire x1="198.12" y1="35.56" x2="203.2" y2="35.56" width="0.1524" layer="91"/>
+</segment>
+</net>
+<net name="N$2" class="0">
+<segment>
+<pinref part="U$8" gate="G$1" pin="P$1"/>
+<wire x1="95.25" y1="20.32" x2="95.25" y2="2.54" width="0.1524" layer="91"/>
+<pinref part="R8" gate="G$1" pin="1"/>
+<wire x1="95.25" y1="2.54" x2="203.2" y2="2.54" width="0.1524" layer="91"/>
+<wire x1="203.2" y1="2.54" x2="203.2" y2="20.32" width="0.1524" layer="91"/>
+</segment>
 </net>
 <net name="N$3" class="0">
 <segment>
 <pinref part="U$3" gate="G$1" pin="P$1"/>
-<wire x1="67.31" y1="50.8" x2="48.26" y2="50.8" width="0.1524" layer="91"/>
-<pinref part="J2" gate="A" pin="1"/>
+<wire x1="67.31" y1="50.8" x2="67.31" y2="43.18" width="0.1524" layer="91"/>
+<pinref part="R3" gate="G$1" pin="1"/>
+<wire x1="67.31" y1="43.18" x2="104.14" y2="43.18" width="0.1524" layer="91"/>
+<wire x1="104.14" y1="43.18" x2="104.14" y2="35.56" width="0.1524" layer="91"/>
 </segment>
 </net>
 <net name="N$4" class="0">
 <segment>
+<pinref part="U$5" gate="G$1" pin="P$1"/>
+<wire x1="67.31" y1="35.56" x2="67.31" y2="27.94" width="0.1524" layer="91"/>
+<wire x1="67.31" y1="27.94" x2="104.14" y2="27.94" width="0.1524" layer="91"/>
+<pinref part="R4" gate="G$1" pin="1"/>
+<wire x1="104.14" y1="27.94" x2="104.14" y2="20.32" width="0.1524" layer="91"/>
+</segment>
+</net>
+<net name="N$5" class="0">
+<segment>
+<pinref part="U$1" gate="G$1" pin="P$1"/>
+<wire x1="67.31" y1="68.58" x2="67.31" y2="83.82" width="0.1524" layer="91"/>
+<pinref part="R5" gate="G$1" pin="1"/>
+<wire x1="67.31" y1="83.82" x2="203.2" y2="83.82" width="0.1524" layer="91"/>
+<wire x1="203.2" y1="83.82" x2="203.2" y2="68.58" width="0.1524" layer="91"/>
+</segment>
+</net>
+<net name="N$6" class="0">
+<segment>
+<pinref part="U$7" gate="G$1" pin="P$1"/>
+<wire x1="67.31" y1="20.32" x2="67.31" y2="12.7" width="0.1524" layer="91"/>
+<wire x1="67.31" y1="12.7" x2="101.6" y2="12.7" width="0.1524" layer="91"/>
+<wire x1="101.6" y1="12.7" x2="101.6" y2="50.8" width="0.1524" layer="91"/>
+<pinref part="R2" gate="G$1" pin="1"/>
+<wire x1="101.6" y1="50.8" x2="104.14" y2="50.8" width="0.1524" layer="91"/>
+</segment>
+</net>
+<net name="N$7" class="0">
+<segment>
 <pinref part="U$4" gate="G$1" pin="P$1"/>
-<pinref part="R2" gate="G$1" pin="1"/>
-<wire x1="95.25" y1="50.8" x2="104.14" y2="50.8" width="0.1524" layer="91"/>
-</segment>
-</net>
-<net name="N$5" class="0">
-<segment>
-<pinref part="U$5" gate="G$1" pin="P$1"/>
-<wire x1="67.31" y1="35.56" x2="48.26" y2="35.56" width="0.1524" layer="91"/>
-<pinref part="J3" gate="A" pin="1"/>
-</segment>
-</net>
-<net name="N$6" class="0">
-<segment>
-<pinref part="U$6" gate="G$1" pin="P$1"/>
-<pinref part="R3" gate="G$1" pin="1"/>
-<wire x1="95.25" y1="35.56" x2="104.14" y2="35.56" width="0.1524" layer="91"/>
-</segment>
-</net>
-<net name="N$7" class="0">
-<segment>
-<pinref part="U$7" gate="G$1" pin="P$1"/>
-<wire x1="67.31" y1="20.32" x2="48.26" y2="20.32" width="0.1524" layer="91"/>
-<pinref part="J4" gate="A" pin="1"/>
-</segment>
-</net>
-<net name="N$8" class="0">
-<segment>
-<pinref part="U$8" gate="G$1" pin="P$1"/>
-<pinref part="R4" gate="G$1" pin="1"/>
-<wire x1="95.25" y1="20.32" x2="104.14" y2="20.32" width="0.1524" layer="91"/>
-</segment>
-</net>
-<net name="N$9" class="0">
-<segment>
-<pinref part="U$9" gate="G$1" pin="P$1"/>
-<wire x1="166.37" y1="68.58" x2="147.32" y2="68.58" width="0.1524" layer="91"/>
-<pinref part="J5" gate="A" pin="1"/>
-</segment>
-</net>
-<net name="N$10" class="0">
-<segment>
-<pinref part="U$10" gate="G$1" pin="P$1"/>
-<pinref part="R5" gate="G$1" pin="1"/>
-<wire x1="194.31" y1="68.58" x2="203.2" y2="68.58" width="0.1524" layer="91"/>
-</segment>
-</net>
-<net name="N$11" class="0">
-<segment>
-<pinref part="U$11" gate="G$1" pin="P$1"/>
-<wire x1="166.37" y1="50.8" x2="147.32" y2="50.8" width="0.1524" layer="91"/>
-<pinref part="J6" gate="A" pin="1"/>
-</segment>
-</net>
-<net name="N$12" class="0">
-<segment>
-<pinref part="U$12" gate="G$1" pin="P$1"/>
-<pinref part="R6" gate="G$1" pin="1"/>
-<wire x1="194.31" y1="50.8" x2="203.2" y2="50.8" width="0.1524" layer="91"/>
-</segment>
-</net>
-<net name="N$13" class="0">
-<segment>
-<pinref part="U$13" gate="G$1" pin="P$1"/>
-<wire x1="166.37" y1="35.56" x2="147.32" y2="35.56" width="0.1524" layer="91"/>
-<pinref part="J7" gate="A" pin="1"/>
-</segment>
-</net>
-<net name="N$14" class="0">
-<segment>
-<pinref part="U$14" gate="G$1" pin="P$1"/>
-<pinref part="R7" gate="G$1" pin="1"/>
-<wire x1="194.31" y1="35.56" x2="203.2" y2="35.56" width="0.1524" layer="91"/>
-</segment>
-</net>
-<net name="N$15" class="0">
-<segment>
-<pinref part="U$15" gate="G$1" pin="P$1"/>
-<wire x1="166.37" y1="20.32" x2="147.32" y2="20.32" width="0.1524" layer="91"/>
-<pinref part="J8" gate="A" pin="1"/>
-</segment>
-</net>
-<net name="N$16" class="0">
-<segment>
-<pinref part="U$16" gate="G$1" pin="P$1"/>
-<pinref part="R8" gate="G$1" pin="1"/>
-<wire x1="194.31" y1="20.32" x2="203.2" y2="20.32" width="0.1524" layer="91"/>
+<wire x1="95.25" y1="50.8" x2="95.25" y2="60.96" width="0.1524" layer="91"/>
+<wire x1="95.25" y1="60.96" x2="104.14" y2="60.96" width="0.1524" layer="91"/>
+<pinref part="R1" gate="G$1" pin="1"/>
+<wire x1="104.14" y1="60.96" x2="104.14" y2="68.58" width="0.1524" layer="91"/>
 </segment>
 </net>
@@
 </drawing>
 <compatibility>
+<note version="8.2" severity="warning">
+Since Version 8.2, EAGLE supports online libraries. The ids
+of those online libraries will not be understood (or retained)
+with this version.
+</note>
 <note version="8.3" severity="warning">
 Since Version 8.3, EAGLE supports URNs for individual library

Commit message: V2 design finished
Connections:
- new net N$10: J6.1, U$11.P$1
- new net N$11: J4.1, U$16.P$1
- new net N$12: J3.1, U$15.P$1
- new net N$13: J7.1, U$14.P$1
- new net N$14: J2.1, U$10.P$1
- new net N$15: J8.1, U$9.P$1
- new net N$16: J1.1, U$13.P$1
- new net N$8: R6.1, U$2.P$1
- new net N$9: J5.1, U$12.P$1
Changed lines of the file:
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@@
+</segment>
+</net>
+<net name="N$8" class="0">
+<segment>
+<pinref part="R6" gate="G$1" pin="1"/>
+<wire x1="203.2" y1="50.8" x2="200.66" y2="50.8" width="0.1524" layer="91"/>
+<wire x1="200.66" y1="50.8" x2="200.66" y2="99.06" width="0.1524" layer="91"/>
+<pinref part="U$2" gate="G$1" pin="P$1"/>
+<wire x1="200.66" y1="99.06" x2="95.25" y2="99.06" width="0.1524" layer="91"/>
+<wire x1="95.25" y1="99.06" x2="95.25" y2="68.58" width="0.1524" layer="91"/>
+</segment>
+</net>
+<net name="N$9" class="0">
+<segment>
+<pinref part="U$12" gate="G$1" pin="P$1"/>
+<wire x1="194.31" y1="50.8" x2="195.58" y2="50.8" width="0.1524" layer="91"/>
+<wire x1="195.58" y1="50.8" x2="195.58" y2="76.2" width="0.1524" layer="91"/>
+<wire x1="195.58" y1="76.2" x2="160.02" y2="76.2" width="0.1524" layer="91"/>
+<wire x1="160.02" y1="76.2" x2="160.02" y2="68.58" width="0.1524" layer="91"/>
+<pinref part="J5" gate="A" pin="1"/>
+<wire x1="160.02" y1="68.58" x2="147.32" y2="68.58" width="0.1524" layer="91"/>
+</segment>
+</net>
+<net name="N$10" class="0">
+<segment>
+<pinref part="U$11" gate="G$1" pin="P$1"/>
+<pinref part="J6" gate="A" pin="1"/>
+<wire x1="166.37" y1="50.8" x2="147.32" y2="50.8" width="0.1524" layer="91"/>
+</segment>
+</net>
+<net name="N$11" class="0">
+<segment>
+<pinref part="U$16" gate="G$1" pin="P$1"/>
+<wire x1="194.31" y1="20.32" x2="194.31" y2="7.62" width="0.1524" layer="91"/>
+<wire x1="194.31" y1="7.62" x2="48.26" y2="7.62" width="0.1524" layer="91"/>
+<pinref part="J4" gate="A" pin="1"/>
+<wire x1="48.26" y1="7.62" x2="48.26" y2="20.32" width="0.1524" layer="91"/>
+</segment>
+</net>
+<net name="N$12" class="0">
+<segment>
+<pinref part="U$15" gate="G$1" pin="P$1"/>
+<wire x1="166.37" y1="20.32" x2="166.37" y2="5.08" width="0.1524" layer="91"/>
+<wire x1="166.37" y1="5.08" x2="50.8" y2="5.08" width="0.1524" layer="91"/>
+<wire x1="50.8" y1="5.08" x2="50.8" y2="35.56" width="0.1524" layer="91"/>
+<pinref part="J3" gate="A" pin="1"/>
+<wire x1="50.8" y1="35.56" x2="48.26" y2="35.56" width="0.1524" layer="91"/>
+</segment>
+</net>
+<net name="N$13" class="0">
+<segment>
+<pinref part="U$14" gate="G$1" pin="P$1"/>
+<wire x1="194.31" y1="35.56" x2="194.31" y2="30.48" width="0.1524" layer="91"/>
+<wire x1="194.31" y1="30.48" x2="147.32" y2="30.48" width="0.1524" layer="91"/>
+<pinref part="J7" gate="A" pin="1"/>
+<wire x1="147.32" y1="30.48" x2="147.32" y2="35.56" width="0.1524" layer="91"/>
+</segment>
+</net>
+<net name="N$14" class="0">
+<segment>
+<pinref part="U$10" gate="G$1" pin="P$1"/>
+<wire x1="194.31" y1="68.58" x2="194.31" y2="86.36" width="0.1524" layer="91"/>
+<wire x1="194.31" y1="86.36" x2="66.04" y2="86.36" width="0.1524" layer="91"/>
+<wire x1="66.04" y1="86.36" x2="66.04" y2="50.8" width="0.1524" layer="91"/>
+<pinref part="J2" gate="A" pin="1"/>
+<wire x1="66.04" y1="50.8" x2="48.26" y2="50.8" width="0.1524" layer="91"/>
+</segment>
+</net>
+<net name="N$15" class="0">
+<segment>
+<pinref part="U$9" gate="G$1" pin="P$1"/>
+<wire x1="166.37" y1="68.58" x2="162.56" y2="68.58" width="0.1524" layer="91"/>
+<wire x1="162.56" y1="68.58" x2="162.56" y2="20.32" width="0.1524" layer="91"/>
+<pinref part="J8" gate="A" pin="1"/>
+<wire x1="162.56" y1="20.32" x2="147.32" y2="20.32" width="0.1524" layer="91"/>
+</segment>
+</net>
+<net name="N$16" class="0">
+<segment>
+<pinref part="U$13" gate="G$1" pin="P$1"/>
+<wire x1="166.37" y1="35.56" x2="165.1" y2="35.56" width="0.1524" layer="91"/>
+<wire x1="165.1" y1="35.56" x2="165.1" y2="104.14" width="0.1524" layer="91"/>
+<wire x1="165.1" y1="104.14" x2="60.96" y2="104.14" width="0.1524" layer="91"/>
+<wire x1="60.96" y1="104.14" x2="60.96" y2="68.58" width="0.1524" layer="91"/>
+<pinref part="J1" gate="A" pin="1"/>
+<wire x1="60.96" y1="68.58" x2="48.26" y2="68.58" width="0.1524" layer="91"/>
 </segment>
 </net>
